File: hardware/ardcore_smd.brd (EAGLE design)
At the start: 40.1 x 100.4 mm, 78 parts, among them IC10 TL072, IC11 74AHCT1G125DBV, IC2 7805DT, IC4 4921, IC5 74AHCT1G125DBV, IC6 ATMEGA328P-AU, IC7 74AHCT1G125DBV, IC8 74AHCT1G125DBV, Y1 RESONATORSMD

Commit message: Changing R50 to 47k to have better gain on output, this was corrected on the Schematics, Board, BOM list and Mouser Project link, also fix in the __dac.setGain(1);__ instruction of the DAC, to use 5v ref instead of 3.3v
Parts:
- R50: value 24.9k -> 47k
Changed lines of the file:
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@@
 <attribute name="VALUE" x="20.835" y="6.855" size="1.016" layer="28" rot="MR180"/>
 </element>
-<element name="R50" library="rcl" package="R0603" value="24.9k" x="27.6" y="1.5" smashed="yes" rot="MR0">
+<element name="R50" library="rcl" package="R0603" value="47k" x="27.6" y="1.5" smashed="yes" rot="MR0">
 <attribute name="NAME" x="28.755" y="2.165" size="1.016" layer="26" rot="MR0"/>
 <attribute name="VALUE" x="23.505" y="1.115" size="0.8128" layer="28" rot="MR180"/>
