File: hardware/v2/ardcore_smd_panel.brd (EAGLE design)
At the start: 40.1 x 100.4 mm, 16 parts

Commit message: changes on panel
Parts:
- removed AUDIO_OUT1, AUDIO_OUT2, CLOCK_IN, CV_A0, CV_A1, CV_A2, CV_A3, DIO4_OUT, DIO5_OUT, DIO6_OUT, DIO7_OUT, RESET: WQP-PJ301M-12_JACK, thonkiconn:WQP-PJ301M-12_JACK
- removed POT_A0, POT_A1, POT_A2, POT_A3: 10k, pot-alps:ALPS_POT_VERTICAL
Connections:
- removed net N$14: RESET.P$2
- removed net N$15: RESET.P$3
- removed net N$6: CV_A3.P$3
Other:
- board size 40.1 x 100.4 mm -> 40 x 100.1 mm
- board text added: "A0"
- board text added: "A1"
- board text added: "A2"
- board text added: "A3"
- board text added: "Ardcore"
- board text added: "CLK"
- board text added: "D0"
- board text added: "D1"
- board text added: "D2"
- board text added: "D3"
- board text added: "O1"
- board text added: "O2"
- board text added: "RST"
Changed lines of the file:
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@@
 <setting verticaltext="up"/>
 </settings>
-<grid distance="0.1" unitdist="mm" unit="mm" style="dots" multiple="1" display="no" altdistance="0.01" altunitdist="mm" altunit="mm"/>
+<grid distance="1" unitdist="mm" unit="mm" style="dots" multiple="1" display="no" altdistance="0.01" altunitdist="mm" altunit="mm"/>
 <layers>
 <layer number="1" name="Top" color="4" fill="1" visible="yes" active="yes"/>
@@
 <layer number="27" name="tValues" color="7" fill="1" visible="yes" active="yes"/>
 <layer number="28" name="bValues" color="7" fill="1" visible="no" active="yes"/>
-<layer number="29" name="tStop" color="7" fill="3" visible="no" active="yes"/>
+<layer number="29" name="tStop" color="7" fill="3" visible="yes" active="yes"/>
 <layer number="30" name="bStop" color="7" fill="6" visible="no" active="yes"/>
 <layer number="31" name="tCream" color="7" fill="4" visible="no" active="yes"/>
@@
 <layer number="44" name="Drills" color="7" fill="1" visible="no" active="yes"/>
 <layer number="45" name="Holes" color="7" fill="1" visible="no" active="yes"/>
-<layer number="46" name="Milling" color="3" fill="1" visible="no" active="yes"/>
+<layer number="46" name="Milling" color="3" fill="1" visible="yes" active="yes"/>
 <layer number="47" name="Measures" color="7" fill="1" visible="no" active="yes"/>
 <layer number="48" name="Document" color="7" fill="1" visible="no" active="yes"/>
@@
 <board>
 <plain>
-<wire x1="40" y1="100" x2="0" y2="100" width="0" layer="20"/>
 <wire x1="0" y1="100" x2="0" y2="0" width="0" layer="20"/>
 <wire x1="0" y1="0" x2="40" y2="0" width="0" layer="20"/>
 <hole x="-14.805" y="30.76" drill="3.2"/>
-<wire x1="39.99" y1="99.97" x2="40.07" y2="-0.36" width="0" layer="20"/>
+<wire x1="39.99" y1="100.07" x2="39.97" y2="-0.06" width="0" layer="20"/>
+<text x="9.2" y="86" size="2.54" layer="1" font="vector" ratio="15">A0</text>
+<circle x="6.2" y="94.5" radius="3.6" width="0.2" layer="46"/>
+<circle x="33.8" y="94.5" radius="3.6" width="0.2" layer="46"/>
+<circle x="6.2" y="63.5" radius="3.6" width="0.2" layer="46"/>
+<circle x="33.8" y="63.5" radius="3.6" width="0.2" layer="46"/>
+<circle x="6.2" y="78.69" radius="3.2" width="0.2" layer="46"/>
+<circle x="33.8" y="77.5" radius="3.2" width="0.2" layer="46"/>
+<circle x="6.2" y="47.5" radius="3.2" width="0.2" layer="46"/>
+<circle x="33.8" y="47.5" radius="3.2" width="0.2" layer="46"/>
+<circle x="4.5" y="21.99" radius="3.2" width="0.2" layer="46"/>
+<circle x="14.833" y="22" radius="3.2" width="0.2" layer="46"/>
+<circle x="25.167" y="22" radius="3.2" width="0.2" layer="46"/>
+<circle x="35.5" y="22" radius="3.2" width="0.2" layer="46"/>
+<circle x="4.5" y="6" radius="3.2" width="0.2" layer="46"/>
+<circle x="14.833" y="6" radius="3.2" width="0.2" layer="46"/>
+<circle x="25.167" y="6" radius="3.2" width="0.2" layer="46"/>
+<circle x="35.5" y="6" radius="3.2" width="0.2" layer="46"/>
+<wire x1="0" y1="100" x2="40" y2="100" width="0" layer="20"/>
+<text x="26.8" y="86" size="2.54" layer="1" font="vector" ratio="15">A1</text>
+<text x="9.2" y="54" size="2.54" layer="1" font="vector" ratio="15">A2</text>
+<text x="26.8" y="54" size="2.54" layer="1" font="vector" ratio="15">A3</text>
+<text x="4.5" y="28" size="2.54" layer="1" font="vector" ratio="15" align="center">D0</text>
+<text x="14.833" y="28" size="2.54" layer="1" font="vector" ratio="15" align="center">D1</text>
+<text x="25.167" y="28" size="2.54" layer="1" font="vector" ratio="15" align="center">D2</text>
+<text x="35.5" y="28" size="2.54" layer="1" font="vector" ratio="15" align="center">D3</text>
+<text x="4.5" y="12" size="2.54" layer="1" font="vector" ratio="15" align="center">CLK</text>
+<text x="14.833" y="12" size="2.54" layer="1" font="vector" ratio="15" align="center">RST</text>
+<text x="25.167" y="12" size="2.54" layer="1" font="vector" ratio="15" align="center">O1</text>
+<text x="35.5" y="12" size="2.54" layer="1" font="vector" ratio="15" align="center">O2</text>
+<circle x="4.5" y="32.42" radius="1.6" width="0.2" layer="46"/>
+<circle x="14.833" y="32.42" radius="1.6" width="0.2" layer="46"/>
+<circle x="25.167" y="32.42" radius="1.6" width="0.2" layer="46"/>
+<circle x="35.5" y="32.42" radius="1.6" width="0.2" layer="46"/>
+<text x="21" y="100" size="3.81" layer="1" font="vector" ratio="15" align="center">Ardcore</text>
+<text x="9.2" y="86" size="2.54" layer="29" font="vector" ratio="15">A0</text>
+<text x="26.8" y="86" size="2.54" layer="29" font="vector" ratio="15">A1</text>
+<text x="26.8" y="54" size="2.54" layer="29" font="vector" ratio="15">A3</text>
+<text x="9.2" y="54" size="2.54" layer="29" font="vector" ratio="15">A2</text>
+<text x="4.5" y="28" size="2.54" layer="29" font="vector" ratio="15" align="center">D0</text>
+<text x="14.833" y="28" size="2.54" layer="29" font="vector" ratio="15" align="center">D1</text>
+<text x="25.167" y="28" size="2.54" layer="29" font="vector" ratio="15" align="center">D2</text>
+<text x="35.5" y="28" size="2.54" layer="29" font="vector" ratio="15" align="center">D3</text>
+<text x="35.5" y="12" size="2.54" layer="29" font="vector" ratio="15" align="center">O2</text>
+<text x="25.167" y="12" size="2.54" layer="29" font="vector" ratio="15" align="center">O1</text>
+<text x="14.833" y="12" size="2.54" layer="29" font="vector" ratio="15" align="center">RST</text>
+<text x="4.5" y="12" size="2.54" layer="29" font="vector" ratio="15" align="center">CLK</text>
+<text x="21" y="100" size="3.81" layer="29" font="vector" ratio="15" align="center">Ardcore</text>
 </plain>
 <attributes>
@@
 </autorouter>
 <elements>
-<element name="POT_A0" library="pot-alps" package="ALPS_POT_VERTICAL" value="10k" x="6.2" y="94.5" rot="R180"/>
-<element name="POT_A1" library="pot-alps" package="ALPS_POT_VERTICAL" value="10k" x="33.8" y="94.5" smashed="yes" rot="R180"/>
-<element name="RESET" library="thonkiconn" package="WQP-PJ301M-12_JACK" value="WQP-PJ301M-12_JACK" x="14.833" y="6" smashed="yes" rot="R180"/>
-<element name="CV_A1" library="thonkiconn" package="WQP-PJ301M-12_JACK" value="WQP-PJ301M-12_JACK" x="33.8" y="78.5" smashed="yes">
-<attribute name="NAME" x="33.2552" y="73.5496" size="0.8128" layer="25" font="vector" rot="R180"/>
-</element>
-<element name="CV_A0" library="thonkiconn" package="WQP-PJ301M-12_JACK" value="WQP-PJ301M-12_JACK" x="6.2" y="78.5" smashed="yes">
-<attribute name="NAME" x="5.4002" y="73.5196" size="0.8128" layer="25" font="vector" rot="R180"/>
-</element>
-<element name="CLOCK_IN" library="thonkiconn" package="WQP-PJ301M-12_JACK" value="WQP-PJ301M-12_JACK" x="4.5" y="6" smashed="yes" rot="R180"/>
-<element name="POT_A2" library="pot-alps" package="ALPS_POT_VERTICAL" value="10k" x="6.2" y="63.5" smashed="yes" rot="R180"/>
-<element name="POT_A3" library="pot-alps" package="ALPS_POT_VERTICAL" value="10k" x="33.8" y="63.5" smashed="yes" rot="R180"/>
-<element name="CV_A3" library="thonkiconn" package="WQP-PJ301M-12_JACK" value="WQP-PJ301M-12_JACK" x="33.8" y="47.5" smashed="yes"/>
-<element name="CV_A2" library="thonkiconn" package="WQP-PJ301M-12_JACK" value="WQP-PJ301M-12_JACK" x="6.2" y="47.5" smashed="yes"/>
-<element name="DIO4_OUT" library="thonkiconn" package="WQP-PJ301M-12_JACK" value="WQP-PJ301M-12_JACK" x="4.5" y="22" smashed="yes" rot="R180"/>
-<element name="DIO5_OUT" library="thonkiconn" package="WQP-PJ301M-12_JACK" value="WQP-PJ301M-12_JACK" x="14.833" y="22" smashed="yes" rot="R180"/>
-<element name="DIO6_OUT" library="thonkiconn" package="WQP-PJ301M-12_JACK" value="WQP-PJ301M-12_JACK" x="25.167" y="22" smashed="yes" rot="R180"/>
-<element name="DIO7_OUT" library="thonkiconn" package="WQP-PJ301M-12_JACK" value="WQP-PJ301M-12_JACK" x="35.5" y="22" smashed="yes" rot="R180"/>
-<element name="AUDIO_OUT1" library="thonkiconn" package="WQP-PJ301M-12_JACK" value="WQP-PJ301M-12_JACK" x="25.167" y="6" smashed="yes" rot="R180"/>
-<element name="AUDIO_OUT2" library="thonkiconn" package="WQP-PJ301M-12_JACK" value="WQP-PJ301M-12_JACK" x="35.5" y="6" smashed="yes" rot="R180"/>
 </elements>
 <signals>
-<signal name="N$14">
-<contactref element="RESET" pad="P$2"/>
-</signal>
-<signal name="N$15">
-<contactref element="RESET" pad="P$3"/>
-</signal>
-<signal name="N$6">
-<contactref element="CV_A3" pad="P$3"/>
-</signal>
 </signals>
 <errors>
