File: hardware/v2/ardcore_smd_panel.sch (EAGLE design)
At the start: 16 parts

Commit message: changes on panel
Parts:
- removed AUDIO_OUT1, AUDIO_OUT2, CLOCK_IN, CV_A0, CV_A1, CV_A2, CV_A3, DIO4_OUT, DIO5_OUT, DIO6_OUT, DIO7_OUT, RESET: WQP-PJ301M-12_JACK, thonkiconn:WQP-PJ301M-12_JACK
- removed POT_A0, POT_A1, POT_A2, POT_A3: 10k, pot-alps:POT_USVERTICAL
Connections:
- removed net N$14: RESET.3
- removed net N$15: RESET.1
- removed net N$6: CV_A3.1
Changed lines of the file:
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@@
 <parts>
 <part name="FRAME1" library="frames" deviceset="A3L-LOC" device=""/>
-<part name="POT_A0" library="pot-alps" deviceset="POT_US" device="VERTICAL" value="10k"/>
-<part name="POT_A1" library="pot-alps" deviceset="POT_US" device="VERTICAL" value="10k"/>
-<part name="RESET" library="thonkiconn" deviceset="WQP-PJ301M-12_JACK" device=""/>
-<part name="CV_A1" library="thonkiconn" deviceset="WQP-PJ301M-12_JACK" device=""/>
-<part name="CV_A0" library="thonkiconn" deviceset="WQP-PJ301M-12_JACK" device=""/>
-<part name="CLOCK_IN" library="thonkiconn" deviceset="WQP-PJ301M-12_JACK" device=""/>
-<part name="POT_A2" library="pot-alps" deviceset="POT_US" device="VERTICAL" value="10k"/>
-<part name="POT_A3" library="pot-alps" deviceset="POT_US" device="VERTICAL" value="10k"/>
-<part name="CV_A3" library="thonkiconn" deviceset="WQP-PJ301M-12_JACK" device=""/>
-<part name="CV_A2" library="thonkiconn" deviceset="WQP-PJ301M-12_JACK" device=""/>
-<part name="DIO4_OUT" library="thonkiconn" deviceset="WQP-PJ301M-12_JACK" device=""/>
-<part name="DIO5_OUT" library="thonkiconn" deviceset="WQP-PJ301M-12_JACK" device=""/>
-<part name="DIO6_OUT" library="thonkiconn" deviceset="WQP-PJ301M-12_JACK" device=""/>
-<part name="DIO7_OUT" library="thonkiconn" deviceset="WQP-PJ301M-12_JACK" device=""/>
-<part name="AUDIO_OUT1" library="thonkiconn" deviceset="WQP-PJ301M-12_JACK" device=""/>
-<part name="AUDIO_OUT2" library="thonkiconn" deviceset="WQP-PJ301M-12_JACK" device=""/>
 </parts>
 <sheets>
@@
 <instances>
 <instance part="FRAME1" gate="G$1" x="0" y="0"/>
-<instance part="POT_A0" gate="G$1" x="147.32" y="213.36"/>
-<instance part="POT_A1" gate="G$1" x="147.32" y="243.84"/>
-<instance part="RESET" gate="G$1" x="40.64" y="205.74" rot="MR0"/>
-<instance part="CV_A1" gate="G$1" x="129.54" y="236.22" rot="MR0"/>
-<instance part="CV_A0" gate="G$1" x="129.54" y="205.74" rot="MR0"/>
-<instance part="CLOCK_IN" gate="G$1" x="40.64" y="241.3" rot="MR0"/>
-<instance part="POT_A2" gate="G$1" x="236.22" y="213.36"/>
-<instance part="POT_A3" gate="G$1" x="236.22" y="238.76"/>
-<instance part="CV_A3" gate="G$1" x="215.9" y="231.14" rot="MR0"/>
-<instance part="CV_A2" gate="G$1" x="215.9" y="208.28" rot="MR0"/>
-<instance part="DIO4_OUT" gate="G$1" x="370.84" y="213.36"/>
-<instance part="DIO5_OUT" gate="G$1" x="370.84" y="187.96"/>
-<instance part="DIO6_OUT" gate="G$1" x="370.84" y="162.56"/>
-<instance part="DIO7_OUT" gate="G$1" x="370.84" y="137.16"/>
 </instances>
 <busses>
 </busses>
 <nets>
-<net name="N$14" class="0">
-<segment>
-<pinref part="RESET" gate="G$1" pin="3"/>
-<wire x1="48.26" y1="205.74" x2="45.72" y2="205.74" width="0.1524" layer="91"/>
-</segment>
-</net>
-<net name="N$15" class="0">
-<segment>
-<pinref part="RESET" gate="G$1" pin="1"/>
-<wire x1="45.72" y1="203.2" x2="48.26" y2="203.2" width="0.1524" layer="91"/>
-</segment>
-</net>
-<net name="N$6" class="0">
-<segment>
-<pinref part="CV_A3" gate="G$1" pin="1"/>
-<wire x1="220.98" y1="228.6" x2="223.52" y2="228.6" width="0.1524" layer="91"/>
-</segment>
-</net>
 </nets>
 </sheet>
@@
 </plain>
 <instances>
-<instance part="AUDIO_OUT1" gate="G$1" x="243.84" y="81.28"/>
-<instance part="AUDIO_OUT2" gate="G$1" x="243.84" y="20.32"/>
 </instances>
 <busses>
