File: hardware/v2/ardcore_smd.brd (EAGLE design)
At the start: 40.1 x 100.4 mm, 78 parts, among them IC10 TL072, IC11 74AHCT1G125DBV, IC2 7805DT, IC4 4921, IC5 74AHCT1G125DBV, IC6 ATMEGA328P-AU, IC7 74AHCT1G125DBV, IC8 74AHCT1G125DBV, Y1 RESONATORSMD

Commit message: New components
Parts:
- removed C21: 100p, rcl:C0603
- removed C29: 47p, rcl:C0603
- removed IC10: TL072, linear:SO08
- removed R45, R46: 39k, rcl:R0603
- removed R50: 47k, rcl:R0603
- removed R55: 1.0k, rcl:R0603
- removed R56: 100k, rcl:R0603
- added AUDIO_OUT1: WQP-PJ301M-12_JACK, thonkiconn:WQP-PJ301M-12_JACK
- added C11: 470n, rcl:C0603
- added C14, C15, C19, C20: 220p, rcl:C0603
- added C17, C23: 18p, rcl:C0603
- added C8, C9: 100n, rcl:C0603
- added IC1, IC3: OPA2171, linear:SO08
- added IC12: LM4040B25, texas:DBZ_R-PDSO-G3
- added IC9: LM4040B10, texas:DBZ_R-PDSO-G3
- added L1: (no value), wuerth-elektronik:0603
- added R12, R14, R17, R22, R24, R26: 39k, rcl:R0603
- added R18, R29: 249k, rcl:R0603
- added R19, R30: 309k, rcl:R0603
- added R20, R31: 1.0k, rcl:R0603
- added R25, R9: 3.3k, rcl:R0603
- added U2: DAC8552IDGKT, Texas Instruments_By_element14_Batch_1:SOP65P490X110-8N
- C22: value 100p -> 470n
- C4: value 10u -> 22u; device rcl:E2,5-5 -> rcl:PANASONIC_C
- IC4: value 4921 -> LM1117-3.3; device adafruit_mcp:SO08 -> og-vreg:SOT223
- moved C22 134.0 mm to (-9.93, -87.5), flipped to the top, turned to 0 degrees
- moved IC4 119.1 mm to (-24.1, -71.5), flipped to the top, turned to 0 degrees
- moved C4 81.2 mm to (-13.6, -69.6), turned to 0 degrees
- moved R3 3.91 mm to (18.4, 67.6)
- moved D1 3.42 mm to (34.0, 98.0)
- moved D2 2.42 mm to (6.00, 98.0)
- moved C1 2.35 mm to (22.4, 67.0)
- moved C7 2.20 mm to (14.9, 67.3), turned to 90 degrees
- moved AVR_ISP 1.21 mm to (14.7, 59.2)
- moved C25 1.12 mm to (24.0, 88.9)
- moved C28 0.83 mm to (25.7, 47.6)
- moved LED3 0.77 mm to (25.2, 32.4)
- moved IC6 0.62 mm to (22.8, 57.6)
- moved C2 0.51 mm to (19.4, 47.8)
- moved C30 0.50 mm to (16.3, 88.6)
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- renumbered AUDIO_OUT to AUDIO_OUT2
Connections:
- removed net N$67: C21.2, C4.+, IC10.6, IC10.7
- removed net N$68: C4.-, R50.2
- removed net N$69: C22.1, IC10.5, R46.1
- removed net N$71: C21.1, R45.1, R46.2
- removed net N$72: AUDIO_OUT2.P$1, R55.1, R56.1
- removed net N$73: C29.2, IC10.1, R55.2
- removed net N$75: C29.1, IC10.2, R50.1, R56.2
- new net +3V3: C4.+, C8.1, IC4.2, L1.1
- new net +3V3_A: C9.1, L1.2, R9.1, U2.1
- new net A: R22.2, U2.4
- new net AREF_-10: C22.1, IC9.2, R19.2, R25.2, R30.2
- new net AREF_2.5: C11.1, IC12.1, R9.2, U2.2
- new net B: R12.2, U2.3
- new net BI_OUT: C17.2, IC1.1, R18.1, R20.2
- new net BI_OUT1: C23.2, IC3.1, R29.1, R31.2
- new net F_CV: C17.1, IC1.2, R17.1, R18.2, R19.1
- new net F_CV1: C23.1, IC3.2, R26.1, R29.2, R30.1
- new net N$1: C14.1, R12.1, R14.2
- new net N$24: C20.1, IC3.5, R24.1
- new net N$26: C19.1, R22.1, R24.2
- new net N$32: AUDIO_OUT1.P$1, R31.1
- new net N$4: C19.2, IC3.6, IC3.7, R26.2
- new net N$42: C14.2, IC1.6, IC1.7, R17.2
- new net N$43: C15.1, IC1.5, R14.1
- net +5V: no longer IC4.1, IC4.6
- net GND: now also AUDIO_OUT1.P$3, C11.2, C15.2, C20.2, C4.-, C8.2, C9.2, IC1.3, IC12.2, IC3.3, IC4.1, IC9.1, U2.8; no longer IC10.3, IC4.5, IC4.7
- net MOSI: no longer IC4.4
- net N$2: now also AUDIO_OUT2.P$1, R20.1; no longer IC4.8, R45.2
- net SCK: no longer IC4.3
- net SS: no longer IC4.2
- net VCC: now also IC1.8, IC3.8, IC4.3; no longer IC10.8
- net VEE: now also IC1.4, IC3.4, R25.1; no longer IC10.4
Routing:
- net GND: track 400.8 -> 0.00 mm, vias 2 -> 0
- net +5V: track 238.0 -> 0.00 mm, vias 9 -> 0
- net SS: track 128.7 -> 0.00 mm, vias 4 -> 0
- net VCC: track 119.8 -> 0.00 mm, vias 1 -> 0
- net VEE: track 110.7 -> 0.00 mm, vias 2 -> 0
- net DIO4: track 98.7 -> 0.00 mm, vias 4 -> 0
- net DIO2: track 96.3 -> 0.00 mm, vias 4 -> 0
- net N$67: track 69.5 -> 0.00 mm, vias 1 -> 0
- net N$73: track 68.1 -> 0.00 mm
- net DIO3: track 66.2 -> 0.00 mm, vias 7 -> 0
- net N$69: track 63.5 -> 0.00 mm, vias 2 -> 0
- net DIO7: track 57.4 -> 0.00 mm, vias 5 -> 0
- net DIO6: track 55.7 -> 0.00 mm, vias 5 -> 0
- net ANI2: track 55.4 -> 0.00 mm, vias 2 -> 0
- net DIO5: track 51.3 -> 0.00 mm, vias 5 -> 0
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
Commit message: removing 3v3 reg
Parts:
- removed C4: 22u, rcl:PANASONIC_C
- removed C8, C9: 100n, rcl:C0603
- removed IC4: LM1117-3.3, og-vreg:SOT223
- R9: value 3.3k -> XXX
Connections:
- removed net +3V3: C4.+, C8.1, IC4.2, L1.1
- removed net +3V3_A: C9.1, L1.2, R9.1, U2.1
- new net N$33: L1.2, R9.1
- net +5V: now also L1.1, U2.1
- net GND: no longer C4.-, C8.2, C9.2, IC4.1
- net VCC: no longer IC4.3

Commit message: almost routed
Parts:
- moved R25 143.9 mm to (38.3, 38.8), flipped to the bottom, turned to 270 degrees
- moved C22 138.7 mm to (37.1, 43.0), flipped to the bottom
- moved IC9 133.7 mm to (36.0, 37.6), flipped to the bottom, turned to 180 degrees
- moved C11 133.7 mm to (32.2, 37.5), flipped to the bottom, turned to 180 degrees
- moved R9 130.6 mm to (1.50, 35.5), flipped to the bottom, turned to 90 degrees
- moved L1 126.8 mm to (8.12, 33.6), flipped to the bottom
- moved IC12 122.6 mm to (2.21, 40.1), flipped to the bottom, turned to 180 degrees
- moved R26 95.1 mm to (20.9, 44.6), flipped to the bottom
- moved R24 92.7 mm to (21.8, 40.6), flipped to the bottom
- moved R12 92.2 mm to (13.0, 48.0), flipped to the bottom, turned to 270 degrees
- moved R14 91.5 mm to (6.69, 48.3), flipped to the bottom
- moved R22 91.1 mm to (9.50, 41.0), flipped to the bottom
- moved R17 87.6 mm to (11.6, 35.6), flipped to the bottom
- moved C23 83.4 mm to (25.1, 34.3), flipped to the bottom, turned to 180 degrees
- moved R29 82.3 mm to (28.9, 34.3), flipped to the bottom, turned to 180 degrees
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Routing:
- net GND: track 0.00 -> 393.9 mm, vias 0 -> 6
- net +5V: track 0.00 -> 217.7 mm, vias 0 -> 11
- net VEE: track 0.00 -> 124.5 mm, vias 0 -> 5
- net VCC: track 0.00 -> 98.6 mm, vias 0 -> 4
- net DIO2: track 0.00 -> 95.2 mm, vias 0 -> 2
- net DIO3: track 0.00 -> 83.9 mm, vias 0 -> 4
- net ANI2: track 0.00 -> 83.0 mm, vias 0 -> 4
- net BI_OUT: track 0.00 -> 51.8 mm, vias 0 -> 2
- net AREF_2.5: track 0.00 -> 51.3 mm, vias 0 -> 4
- net AREF_-10: track 0.00 -> 38.1 mm, vias 0 -> 2
- net BI_OUT1: track 0.00 -> 36.1 mm, vias 0 -> 4
- net ANI4: track 0.00 -> 36.1 mm, vias 0 -> 2
- net RESET: track 0.00 -> 30.5 mm, vias 0 -> 2
- net F_CV1: track 0.00 -> 29.7 mm, vias 0 -> 2
- net F_CV: track 0.00 -> 28.4 mm
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
Commit message: Adding version
Parts:
- IC12: value LM4040B25 -> LM4040
- IC9: value LM4040B10 -> LM4040
- U2: value DAC8552IDGKT -> DAC8552
Routing:
- net DIO4: track 18.3 -> 77.6 mm, vias 2 -> 4
- net DIO7: track 20.2 -> 75.0 mm, vias 2 -> 4
- net DIO6: track 17.8 -> 55.3 mm
- net DIO5: track 18.5 -> 54.4 mm, vias 2 -> 4
- net GND: track 393.9 -> 427.4 mm, vias 6 -> 7
- net VCC: track 98.6 -> 111.1 mm
- net +5V: track 217.7 -> 228.5 mm
Other:
- board text removed: "Original Ardcore by 20objects.com"
- board text removed: "PCBLayout by luix and gb github.com/ttreintaysiete"
- board text removed: "booty"
- board text removed: "bulbasaur?"
- board text removed: "egghead"
- board text removed: "its a trap!!!!111"
- board text removed: "pipsqueak"
- board text removed: "reflow the SMT"
- board text removed: "splendiferous"

Commit message: Adding v2 fixed gerbers
Connections:
- net MOSI: now also U2.7
- net SCK: now also U2.6
- net SS: now also U2.5
Routing:
- net SS: track 0.00 -> 66.4 mm, vias 0 -> 4
- net MOSI: track 7.30 -> 51.6 mm, vias 0 -> 5
- net SCK: track 8.78 -> 46.3 mm, vias 1 -> 5
- net +5V: track 228.5 -> 230.4 mm
